Commit message: Changed robot shape

File: urdf/my_robot.xacro (robot description, xacro)
@@ -1,4 +1,3 @@
 <?xml version='1.0'?>
-<!--Drive robot straight, might be swaying one direction a little bit more-->
 <robot name="my_robot" xmlns:xacro="http://www.ros.org/wiki/xacro">
   <xacro:include filename="$(find localization)/urdf/my_robot.gazebo"/>
@@ -17,13 +16,13 @@
   <link name="robot_footprint"></link>
   <joint name="robot_footprint_joint" type="fixed">
-    <origin xyz="0 0 0" rpy="0 0 0" />
-    <parent link="robot_footprint"/>
-    <child link="chassis" />
+  <origin xyz="0 0 0" rpy="0 0 0" />
+  <parent link="robot_footprint"/>
+  <child link="chassis" />
   </joint>
   <link name='chassis'>
-      <pose>0 0 0.1 0 0 0</pose>
+      <pose>0 0 0.15 0 0 0</pose>
       <inertial>
         <mass value="15.0"/>
-        <origin xyz="0.0 0 0.05" rpy=" 0 0 0"/>
+        <origin xyz="0.0 0 0" rpy=" 0 0 0"/>
         <inertia
                 ixx="0.1" ixy="0" ixz="0"
@@ -33,5 +32,5 @@
       </inertial>
       <collision name='collision'>
-        <origin xyz="0 0 0.05" rpy="0 0 0"/>
+        <origin xyz="0 0 0" rpy=" 0 0 0"/>
         <geometry>
               <cylinder radius="0.35" length="0.15"/>
@@ -39,41 +38,35 @@
       </collision>
       <visual name='chassis_visual'>
-        <origin xyz="0 0 0.05" rpy="0 0 0"/>
+        <origin xyz="0 0 0" rpy=" 0 0 0"/>
         <geometry>
               <cylinder radius="0.35" length="0.15"/>
         </geometry>
         <material name="green">
-          <color rgba="0.1 0.8 0.2 1"/>
+          <color rgba="0.1 0.0 0.2 1"/>
         </material>
       </visual>
-      <collision name="front_caster_collision">
-        <origin xyz="0.25 0 0" rpy="0 0 0"/>
-        <geometry>
-            <sphere radius="0.075"/>
+      <collision name='back_caster_collision'>
+        <origin xyz="-0.25 0 -0.05" rpy=" 0 0 0"/>
+        <geometry>
+              <sphere radius="0.0499"/>
         </geometry>
       </collision>
-      <visual name="front_caster_visual">
-        <origin xyz="0.25 0 0" rpy="0 0 0"/>
-        <geometry>
-            <sphere radius="0.075"/>
-        </geometry>
-        <material name="grey">
-          <color rgba="0.5 0.6 0.7 1"/>
-        </material>
+      <visual name='back_caster_visual'>
+        <origin xyz="-0.25 0 -0.05" rpy=" 0 0 0"/>
+        <geometry>
+              <sphere radius="0.05"/>
+        </geometry>
       </visual>
-      <collision name="back_caster_collision">
-        <origin xyz="-0.25 0 0" rpy="0 0 0"/>
-        <geometry>
-            <sphere radius="0.075"/>
+      <collision name='front_caster_collision'>
+        <origin xyz="0.25 0 -0.05" rpy=" 0 0 0"/>
+        <geometry>
+              <sphere radius="0.0499"/>
         </geometry>
       </collision>
-      <visual name="back_caster_visual">
-        <origin xyz="-0.25 0 0" rpy="0 0 0"/>
-        <geometry>
-            <sphere radius="0.075"/>
-        </geometry>
-        <material name="grey">
-          <color rgba="0.5 0.6 0.7 1"/>
-        </material>
+      <visual name='front_caster_visual'>
+        <origin xyz="0.25 0 -0.05" rpy=" 0 0 0"/>
+        <geometry>
+              <sphere radius="0.05"/>
+        </geometry>
       </visual>
   </link>
@@ -92,17 +85,19 @@
       <origin xyz="0 0 0" rpy="0 1.5707 1.5707"/>
         <geometry>
-          <cylinder radius="0.075" length="0.05"/>
-        </geometry>
-      <material name="black"/>
+          <cylinder radius="0.1" length="0.05"/>
+        </geometry>
+        <material name="black">
+          <color rgba="0.0 0.0 0.0 1.0"/>
+        </material>
     </visual>
     <collision name="left_wheel_collision">
       <origin xyz="0 0 0" rpy="0 1.5707 1.5707"/>
         <geometry>
-          <cylinder radius="0.075" length="0.05"/>
+          <cylinder radius="0.1" length="0.05"/>
         </geometry>
     </collision>
 	</link>
   <joint type="continuous" name="left_wheel_hinge">
-    <origin xyz="-0.05 0.3 0" rpy="0 0 0"/>
+    <origin xyz="0 0.25 0" rpy="0 0 0"/>
     <child link="left_wheel"/>
     <parent link="chassis"/>
@@ -125,8 +120,8 @@
         <origin xyz="0 0 0" rpy="0 1.5707 1.5707"/>
         <geometry>
-            <cylinder radius="0.075" length="0.05"/>
+            <cylinder radius="0.1" length="0.05"/>
         </geometry>
         <material name="black">
-          <color rgba="0 0 0 1"/>
+          <color rgba="0.0 0.0 0.0 1.0"/>
         </material>
     </visual>
@@ -134,10 +129,10 @@
         <origin xyz="0 0 0" rpy="0 1.5707 1.5707"/>
         <geometry>
-            <cylinder radius="0.075" length="0.05"/>
+            <cylinder radius="0.1" length="0.05"/>
         </geometry>
     </collision>
   </link>
   <joint type="continuous" name="right_wheel_hinge">
-    <origin xyz="-0.05 -0.3 0" rpy="0 0 0"/>
+    <origin xyz="0 -0.25 0" rpy="0 0 0"/>
     <child link="right_wheel"/>
     <parent link="chassis"/>
@@ -174,5 +169,5 @@
   </link>
   <joint type="fixed" name="camera_joint">
-    <origin xyz="0.35 0 0.025" rpy="0 0 0"/>
+    <origin xyz="0.35 0 0" rpy="0 0 0"/>
     <child link="camera"/>
     <parent link="chassis"/>
@@ -204,5 +199,5 @@
   </link>
   <joint type="fixed" name="hokuyo_joint">
-    <origin xyz="0.0 0 0.15" rpy="0 0 0"/>
+    <origin xyz="0.15 0 0.1" rpy="0 0 0"/>
     <child link="hokuyo"/>
     <parent link="chassis"/>
